Commit message: add orb_slam with odom test tool

File: my_robot.urdf (robot description, URDF)
Before this commit: robot myRobot, 22 links, 21 joints
Joints:
- joint camera_sensor_left_joint: origin xyz=0.175 0.05 0.005 rpy=0 0 0 -> xyz=0.175 0.05 0.005 rpy=0 -1.5708 0
- joint camera_sensor_right_joint: origin xyz=0.175 -0.05 0.005 rpy=0 0 0 -> xyz=0.175 -0.05 0.005 rpy=0 -1.5708 0
